Commit message: Changed lidar to 3d_lidar

File: urdf/actor-1.urdf (robot description, URDF)
Before this commit: robot ltu-actor, 9 links, 8 joints
Links:
- removed link lidar
- added link 3d_lidar; visual cylinder length=0.03 radius=0.025
Joints:
- removed joint camera_to_lidar
- added joint camera_to_3d_lidar: type fixed, parent camera, child 3d_lidar, origin xyz=0 0 0.13

Commit message: Added 2d lidars and minor changes

File: urdf/actor-1.urdf (robot description, URDF)
Before this commit: robot ltu-actor, 9 links, 8 joints
Links:
- removed link 3d_lidar
- removed link camera
- added link front_2d_lidar; visual cylinder length=0.08 radius=0.03
- added link front_camera; visual box size=0.05 0.05 0.05
- added link rear_2d_lidar; visual cylinder length=0.08 radius=0.03
- added link top_3d_lidar; visual cylinder length=0.072 radius=0.05
- link base_link: geometry visual cylinder length=1.38 radius=0.1
- link body: geometry visual box size=2.6 1.30 1.6
- link front_axle: geometry visual cylinder length=1.38 radius=0.1
- link front_left_wheel: geometry visual cylinder length=0.2 radius=0.28
- link front_right_wheel: geometry visual cylinder length=0.2 radius=0.28
- link rear_left_wheel: geometry visual cylinder length=0.2 radius=0.28
- link rear_right_wheel: geometry visual cylinder length=0.2 radius=0.28
Joints:
- removed joint body_to_camera
- removed joint camera_to_3d_lidar
- added joint body_to_front_2d_lidar: type fixed, parent body, child front_2d_lidar, origin xyz=1.74 0 -1.4
- added joint body_to_front_camera: type fixed, parent body, child front_camera, origin xyz=0.56 0 0.03
- added joint body_to_rear_2d_lidar: type fixed, parent body, child rear_2d_lidar, origin xyz=-0.94 0 -1.4
- added joint camera_to_top_3d_lidar: type fixed, parent front_camera, child top_3d_lidar, origin xyz=0 0 0.09

Commit message: Turned rear 2d lidar 180

File: urdf/actor-1.urdf (robot description, URDF)
Before this commit: robot ltu-actor, 11 links, 10 joints
Joints:
- joint body_to_rear_2d_lidar: origin xyz=-0.94 0 -1.4 -> xyz=-0.94 0 -1.4 rpy=0 0 1.57075

Commit message: Rotate rear_2d_lidar 180

File: urdf/actor-1.urdf (robot description, URDF)
Before this commit: robot ltu-actor, 11 links, 10 joints
Joints:
- joint body_to_rear_2d_lidar: origin xyz=-0.94 0 -1.4 rpy=0 0 1.57075 -> xyz=-0.94 0 -1.4 rpy=0 0 3.14159

Commit message: Flipped read lidar upside down

File: urdf/actor-1.urdf (robot description, URDF)
Before this commit: robot ltu-actor, 11 links, 10 joints
Joints:
- joint body_to_rear_2d_lidar: origin xyz=-0.94 0 -1.4 rpy=0 0 3.14159 -> xyz=-0.94 0 -1.4 rpy=3.14159 0 3.14159
